File: Tracker.sch (EAGLE design)
At the start: 37 parts, among them IC2 74AHC1G125DBV, IC3 74AHC1G125DBV, M1 HX1, X1 BU-SMA-V

Commit message: rev2
Removed .x#h files, removed teaching examples, shrunk footprint, made project library
Parts:
- removed JP4: (no value), SparkFun:M06POLAR
- removed U$12: CKN10160-ND, SHC:CKN10160-ND
- removed U$9: AVR-PDIVERT, avr-7:AVR-PDIVERT
- added LOG: LOG, Tracker:SPARKFUN_M06SIP
- added PDI: AVR-7_AVR-PDIVERT, Tracker:AVR-7_AVR-PDIVERT
- added SWITCH: (no value), switch:M251
- L1: value 10uH -> FB_0402; device rcl:L-USL2012C -> rc-master-smd:FB_0402
- L3: value FB_0402 -> 10uH; device rc-master-smd:FB_0402 -> rcl:L-USL2012C
- renumbered IC1 to MCU, IC2 to LOG1, IC3 to LOG2, LED1 to LED, U$1 to MS5607, U$10 to 3.3REG, U$11 to 5.0REG, U$2 to GPS, U$3 to BATT2, U$4 to BATT1
Connections:
- removed net N$11: DIODE.C, U$12.NC
- removed net N$17: C15.2, C16.2, L2.1, MCU.AVCC
- new net AVCC: C15.2, C16.2, L4.1, MCU.AVCC
- new net N$7: DIODE.C, SWITCH.O
- net BATT: now also SWITCH.P; no longer U$12.COM
- net GND: now also LOG.5, PDI.6; no longer JP4.5, U$9.6
- net N$1: now also L1.2; no longer L3.2
- net N$18: now also L3.1, L4.2; no longer L1.1, L2.2
- net N$2: now also L2.2; no longer L4.2
- net PDI-CLK: now also PDI.5; no longer U$9.5
- net PDI-DATA: now also PDI.1; no longer U$9.1
- net RXC: now also L1.1; no longer L3.1
- net RXD: now also LOG.3; no longer JP4.3
- net TXC: now also L2.1; no longer L4.1
- net TXD: now also LOG.2; no longer JP4.2
- net VCC: now also L3.2, LOG.4, PDI.2; no longer JP4.4, L1.2, U$9.2
Other:
- moved on the sheet: L1, L2, L3, L4
